File: PiCoCo/PiCoCo.kicad_sch (KiCad schematic)
At the start: 6 parts, among them J1 Conn_01x02_Pin, U1 Pico, U2 74HC244, U3 74HC244

Commit message: Updated schematic
Parts:
- P1: footprint CoCoEPROMpak:COCO-CART-2.1X1.75 -> PiCoCo:COCO-CART-2.1X1.75
- U1: footprint RPi_Pico:RPi_Pico_SMD_TH -> PiCoCo:RPi_Pico_SMD_TH; symbol MCU_RaspberryPi_and_Boards:Pico -> PiCoCo:Pico
Connections:
- net GND: now also U2.1 (1OE), U2.19 (2OE), U3.1 (1OE), U3.19 (2OE); no longer P1.34 (GND@2)
- net A3: now reaches U2.11 (2A3)
- net A3: now also P1.22 (A3)
- net GPIO11: now reaches U2.12 (1Y3)
- net GPIO11: now also U1.15 (GPIO11)
- net A2: now reaches U2.13 (2A2)
- net A2: now also P1.21 (A2)
- net GPIO10: now reaches U2.14 (1Y2)
- net GPIO10: now also U1.14 (GPIO10)
- net A1: now reaches U2.15 (2A1)
- net A1: now also P1.20 (A1)
- net GPIO9: now reaches U2.16 (1Y1)
- net GPIO9: now also U1.12 (GPIO9)
- net A0: now reaches U2.17 (2A0)
- net A0: now also P1.19 (A0)
- net GPIO8: now reaches U2.18 (1Y0)
- net GPIO8: now also U1.11 (GPIO8)
- net GPIO12: now reaches U2.3 (2Y0)
- net GPIO12: now also U1.16 (GPIO12)
- net GPIO13: now reaches U2.5 (2Y1)
- net GPIO13: now also U1.17 (GPIO13)
- net E_CLK: now reaches U2.6 (1A2)
- net E_CLK: now also P1.6 (E)
- net GPIO14: now reaches U2.7 (2Y2)
- net GPIO14: now also U1.19 (GPIO14)
- net ~{RW}: now reaches U2.8 (1A3)
- net ~{RW}: now also P1.18 (R/~{W})
- net GPIO15: now reaches U2.9 (2Y3)
- net GPIO15: now also U1.20 (GPIO15)
- net SCS renamed ~{SCS}
- no-connect marks 3 -> 39

Commit message: Updated 12_13
Parts:
- added IC1, IC2: 74FST3257DR2G, SOIC127P600X175-16N, symbol PiCoCo:74FST3257DR2G
Connections:
- net 3V: now also IC1.16 (VCC), IC2.16 (VCC)
- net A0: now also IC1.2 (1B1); no longer U2.17 (2A0)
- net A1: now also IC1.5 (2B1); no longer U2.15 (2A1)
- net A2: now also IC1.14 (4B1); no longer U2.13 (2A2)
- net A3: now also IC1.11 (3B1); no longer U2.11 (2A3)
- net D0: now also IC1.3 (1B2); no longer U3.2 (1A0)
- net D1: now also IC1.6 (2B2); no longer U3.4 (1A1)
- net D2: now also IC1.13 (4B2); no longer U3.6 (1A2)
- net D3: now also IC1.10 (3B2); no longer U3.8 (1A3)
- net D4: now also IC2.3 (1B2); no longer U3.17 (2A0)
- net D5: now also IC2.6 (2B2); no longer U3.15 (2A1)
- net D6: now also IC2.13 (4B2); no longer U3.13 (2A2)
- net D7: now also IC2.10 (3B2); no longer U3.11 (2A3)
- net E_CLK: now also U2.4 (1A1); no longer U2.6 (1A2)
- net GND: now also IC1.15 (~{OE}), IC1.8 (GND), IC2.15 (~{OE}), IC2.8 (GND)
- net Q_CLK: now also U2.2 (1A0); no longer U2.4 (1A1)
- net ~{RW}: now also U2.6 (1A2); no longer U2.8 (1A3)
- net A4: now reaches P1.23 (A4)
- net A4: now also IC2.2 (1B1)
- net A5: now reaches P1.24 (A5)
- net A5: now also IC2.5 (2B1)
- net A6: now reaches P1.25 (A6)
- net A6: now also IC2.14 (4B1)
- net A7: now reaches P1.26 (A7)
- net A7: now also IC2.11 (3B1)
- net A8: now reaches P1.27 (A8)
- net A8: now also U3.2 (1A0)
- net A9: now reaches P1.28 (A9)
- net A9: now also U3.4 (1A1)
- net A10: now reaches P1.29 (A10)
- net A10: now also U3.6 (1A2)
- net ~{HALT}: now reaches P1.3 (~{HALT})
- net ~{HALT}: now also U2.13 (2A2)
- net A11: now reaches P1.30 (A11)
- net A11: now also U3.8 (1A3)
- net A12: now reaches P1.31 (A12)
- net A12: now also U3.17 (2A0)
- net A13: now reaches P1.37 (A13)
- net A13: now also U3.15 (2A1)
- net A14: now reaches P1.38 (A14)
- net A14: now also U3.13 (2A2)
- net A15: now reaches P1.39 (A15)
- net A15: now also U3.11 (2A3)
- net ~{NMI}: now reaches P1.4 (~{NMI})
- net ~{NMI}: now also U2.15 (2A1)
- net ~{SLENB}: now reaches P1.40 (~{SLENB})
- net ~{SLENB}: now also U2.8 (1A3)
- net ~{RESET}: now reaches P1.5 (~{RESET})
- net ~{RESET}: now also U2.17 (2A0)
- net SEL: now reaches U1.21 (GPIO16)
- net SEL: now also IC1.1 (S), IC2.1 (S)
- net Q_GCLK: now reaches U1.22 (GPIO17)
- net Q_GCLK: now also U2.18 (1Y0)
- net E_GCLK: now reaches U1.24 (GPIO18)
- net E_GCLK: now also U2.16 (1Y1)
- net ~{GRW}: now reaches U1.25 (GPIO19)
- net ~{GRW}: now also U2.14 (1Y2)
- net ~{GSLENB}: now reaches U1.26 (GPIO20)
- net ~{GSLENB}: now also U2.12 (1Y3)
- net ~{GRESET}: now reaches U1.27 (GPIO21)
- net ~{GRESET}: now also U2.3 (2Y0)
- net ~{GNMI}: now reaches U1.29 (GPIO22)
- net ~{GNMI}: now also U2.5 (2Y1)
- net ~{GHALT}: now reaches U1.31 (GPIO26_ADC0)
- net ~{GHALT}: now also U2.7 (2Y2)
- net GPIO0 renamed AD0
- net AD0: now also IC1.4 (1A); no longer U3.18 (1Y0)
- net GPIO1 renamed AD1
- net AD1: now also IC1.7 (2A); no longer U3.16 (1Y1)
- net GPIO10 renamed AG10
- net AG10: now also U3.14 (1Y2); no longer U2.14 (1Y2)
- net GPIO11 renamed AG11
- net AG11: now also U3.12 (1Y3); no longer U2.12 (1Y3)
- net GPIO12 renamed AG12
- net AG12: now also U3.3 (2Y0); no longer U2.3 (2Y0)
- net GPIO13 renamed AG13
- net AG13: now also U3.5 (2Y1); no longer U2.5 (2Y1)
- net GPIO14 renamed AG14
- net AG14: now also U3.7 (2Y2); no longer U2.7 (2Y2)
- net GPIO15: no longer names the net of U2.9 (2Y3)
- net GPIO15: no longer U1.20 (GPIO15)
- net GPIO2 renamed AD2
- net AD2: now also IC1.12 (4A); no longer U3.14 (1Y2)
- net GPIO3 renamed AD3
- net AD3: now also IC1.9 (3A); no longer U3.12 (1Y3)
- net GPIO4 renamed AD4
- net AD4: now also IC2.4 (1A); no longer U3.3 (2Y0)
- net GPIO5 renamed AD5
- net AD5: now also IC2.7 (2A); no longer U3.5 (2Y1)
- net GPIO6 renamed AD6
- net AD6: now also IC2.12 (4A); no longer U3.7 (2Y2)
- net GPIO7 renamed AD7
- net AD7: now also IC2.9 (3A); no longer U3.9 (2Y3)
- net GPIO8 renamed AG8
- net AG8: now also U3.18 (1Y0); no longer U2.18 (1Y0)
- net GPIO9 renamed AG9
- net AG9: now also U3.16 (1Y1); no longer U2.16 (1Y1)
- net ~{SCS}: no longer names the net of P1.36 (~{SCS})
- net ~{SCS}: no longer U2.2 (1A0)
- new net AG15: U1.20 (GPIO15), U3.9 (2Y3)
- no-connect marks 39 -> 18

Commit message: Updated initial PCB
Parts:
- added C1, C2, C3, C4, C5: .1U, Capacitor_SMD:C_0201_0603Metric_Pad0.64x0.40mm_HandSolder, symbol Device:C
- added R1: 10k, Resistor_SMD:R_0201_0603Metric_Pad0.64x0.40mm_HandSolder, symbol Device:R
- added U4: 74HC244, Package_SO:TSSOP-20_4.4x6.5mm_P0.65mm, symbol 74xx:74HC244
- IC1, IC2: footprint SOIC127P600X175-16N -> Package_SO:TSSOP-16_4.4x5mm_P0.65mm
Connections:
- net +5V: now also U2.20 (VCC), C1.2
- net 3V: now also C2.2, C3.2, C4.2, C5.2, R1.1, U4.20 (VCC); no longer U2.20 (VCC)
- net E_CLK: now also U4.4 (1A1); no longer U2.4 (1A1)
- net E_GCLK: now also U4.16 (1Y1); no longer U2.16 (1Y1)
- net GND: now also U2.11 (2A3), U2.13 (2A2), U2.15 (2A1), U2.17 (2A0), C1.1, C2.1, C3.1, C4.1, C5.1, U4.10 (GND), U4.11 (2A3), U4.13 (2A2), U4.15 (2A1), U4.17 (2A0), U4.8 (1A3); no longer IC1.15 (~{OE}), IC2.15 (~{OE}), U2.1 (1OE), U2.19 (2OE), U3.1 (1OE), U3.19 (2OE)
- net Q_CLK: now also U4.2 (1A0); no longer U2.2 (1A0)
- net Q_GCLK: now also U4.18 (1Y0); no longer U2.18 (1Y0)
- net ~{GHALT}: now also U2.4 (1A1); no longer U2.7 (2Y2)
- net ~{GNMI}: now also U2.6 (1A2); no longer U2.5 (2Y1)
- net ~{GRESET}: now also U2.8 (1A3); no longer U2.3 (2Y0)
- net ~{GRW}: now also U4.14 (1Y2); no longer U2.14 (1Y2)
- net ~{GSLENB}: now also U2.2 (1A0); no longer U2.12 (1Y3)
- net ~{HALT}: now also U2.16 (1Y1); no longer U2.13 (2A2)
- net ~{NMI}: now also U2.14 (1Y2); no longer U2.15 (2A1)
- net ~{RESET}: now also U2.12 (1Y3); no longer U2.17 (2A0)
- net ~{RW}: now also U4.6 (1A2); no longer U2.6 (1A2)
- net ~{SLENB}: now also U2.18 (1Y0); no longer U2.8 (1A3)
- net ~{CART}: now reaches J1.1 (Pin_1), P1.8 (~{CART})
- net EN: now reaches U1.34 (GPIO28_ADC2)
- net EN: now also IC1.15 (~{OE}), IC2.15 (~{OE}), U2.1 (1OE), U2.19 (2OE), U3.1 (1OE), U3.19 (2OE), R1.2, U4.1 (1OE), U4.19 (2OE)
- no-connect marks 18 -> 24
Other:
- moved on the sheet: U2

Commit message: Cleanup
Parts:
- C1, C2, C3, C4, C5: footprint Capacitor_SMD:C_0201_0603Metric_Pad0.64x0.40mm_HandSolder -> Capacitor_SMD:C_0805_2012Metric_Pad1.18x1.45mm_HandSolder
- R1: footprint Resistor_SMD:R_0201_0603Metric_Pad0.64x0.40mm_HandSolder -> Resistor_SMD:R_0805_2012Metric_Pad1.20x1.40mm_HandSolder
Connections:
- no-connect marks 24 -> 23
Changed lines of the file:
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@@
   (no_connect (at 172.974 65.024))
   (no_connect (at 54.61 125.222))
-  (no_connect (at 57.15 125.222))
   (no_connect (at 222.504 90.678))
   (no_connect (at 59.69 28.702))
@@
     (pin "17")
     (pin "35")
-    (pin "MTG2")
     (pin "11")
     (pin "6")
@@
       (effects (font (size 1.27 1.27)))
     )
-    (property "Footprint" "Capacitor_SMD:C_0201_0603Metric_Pad0.64x0.40mm_HandSolder" (at 113.538 26.1112 0)
+    (property "Footprint" "Capacitor_SMD:C_0805_2012Metric_Pad1.18x1.45mm_HandSolder" (at 113.538 26.1112 0)
       (effects (font (size 1.27 1.27)) hide)
     )
@@
       (effects (font (size 1.27 1.27)))
     )
-    (property "Footprint" "Capacitor_SMD:C_0201_0603Metric_Pad0.64x0.40mm_HandSolder" (at 107.442 157.4292 0)
+    (property "Footprint" "Capacitor_SMD:C_0805_2012Metric_Pad1.18x1.45mm_HandSolder" (at 107.442 157.4292 0)
       (effects (font (size 1.27 1.27)) hide)
     )
@@
       (effects (font (size 1.27 1.27)) (justify left))
     )
-    (property "Footprint" "Resistor_SMD:R_0201_0603Metric_Pad0.64x0.40mm_HandSolder" (at 261.366 48.006 90)
+    (property "Footprint" "Resistor_SMD:R_0805_2012Metric_Pad1.20x1.40mm_HandSolder" (at 261.366 48.006 90)
       (effects (font (size 1.27 1.27)) hide)
     )
@@
       (effects (font (size 1.27 1.27)))
     )
-    (property "Footprint" "Capacitor_SMD:C_0201_0603Metric_Pad0.64x0.40mm_HandSolder" (at 64.516 157.6832 0)
+    (property "Footprint" "Capacitor_SMD:C_0805_2012Metric_Pad1.18x1.45mm_HandSolder" (at 64.516 157.6832 0)
       (effects (font (size 1.27 1.27)) hide)
     )
@@
       (effects (font (size 1.27 1.27)))
     )
-    (property "Footprint" "Capacitor_SMD:C_0201_0603Metric_Pad0.64x0.40mm_HandSolder" (at 165.1 35.7632 0)
+    (property "Footprint" "Capacitor_SMD:C_0805_2012Metric_Pad1.18x1.45mm_HandSolder" (at 165.1 35.7632 0)
       (effects (font (size 1.27 1.27)) hide)
     )
@@
       (effects (font (size 1.27 1.27)))
     )
-    (property "Footprint" "Capacitor_SMD:C_0201_0603Metric_Pad0.64x0.40mm_HandSolder" (at 148.336 106.1212 0)
-      (effects (font (size 1.27 1.27)) hide)
-    )
+    (property "Footprint" "Capacitor_SMD:C_0805_2012Metric_Pad1.18x1.45mm_HandSolder" (at 148.336 106.1212 0)
+      (effects (font (size 1.27 1.27)) hide)
+    )
