File: PiCoCo/PiCoCo.kicad_pcb (KiCad board)
At the start: 2 copper layers, 98 x 77.2 mm, 63 parts, among them J1 EXP (Plus-W), P1 COCO-CART, Q2 2N7002, Q3 2N7002, Q4 2N7002, U1 Pico 2 / RP2350B-Plus-W, U10 SN74LVC245A, U11 SN74LVC245A, U12 SN74LVC245A, U13 SN74LVC245A, U14 AMS1117-3.3, U15 SN74LVC00A

Commit message: v2.3.1: J2/J3 DNP 1x3 pin-header twins of JP3/JP5 (movable shunt option)
Same nets as the solder jumpers; fit at most one of each pair. Re-routed;
DRC 0 errors / 0 unconnected / 0 parity; GND coverage under the bus 40%
(was 27%). BOM/CPL unchanged (17 lines / 38 parts, headers are DNP).

Co-Authored-By: Claude Fable 5.1 <noreply@anthropic.com>
Claude-Session: https://claude.ai/code/session_013jbrP69zFzwzxjawTKy2c7
Parts:
- added J2: JP3 hdr, Connector_PinHeader_2.54mm:PinHeader_1x03_P2.54mm_Vertical, F.Cu at (170.0, 56.0)
- added J3: JP5 hdr, Connector_PinHeader_2.54mm:PinHeader_1x03_P2.54mm_Vertical, F.Cu at (131.0, 61.0)
Routing:
- net SLENB_BUF: track 99.6 -> 74.1 mm, vias 6 -> 2
- net NMI_DRV: track 55.9 -> 80.3 mm
- net RW_BUF: track 134.3 -> 111.9 mm, vias 3 -> 2
- net RESET_CART: track 81.9 -> 98.6 mm, vias 2 -> 6
- net GND: track 536.8 -> 552.5 mm, vias 60 -> 63
- net A14_BUF: track 103.7 -> 119.2 mm, vias 18 -> 8
- net A10_BUF: track 85.2 -> 72.1 mm
- net A15_BUF: track 95.8 -> 82.9 mm, vias 4 -> 2
- net OE_FW: track 42.2 -> 54.7 mm
- net Q_CART: track 102.9 -> 90.8 mm, vias 6 -> 4
- net A9_BUF: track 78.1 -> 66.0 mm
- net CTS_BUF: track 126.7 -> 114.7 mm
- net EXP_GP45: track 57.4 -> 45.5 mm
- net D7: track 73.3 -> 61.6 mm, vias 2 -> 1
- net D5: track 58.1 -> 68.2 mm
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Other:
- board text added: "(JP3/J2 or JP5/J3, never both)"
- board text added: "JP3/J2 1-2=AUDIO"
- board text added: "JP5/J3: hdr34-> 1-2 /CART 2-3 /NMI"
- board text removed: "(JP3 or JP5, never both)"
- board text removed: "JP3 1-2=AUDIO"
- board text removed: "JP5: hdr34-> 1-2 /CART 2-3 /NMI"

Commit message: v2.4: board cutout so a Waveshare RP2350B-Plus-W mounts flat
The Plus-W carries its 16 MB flash (W25Q128JVSIQ, SOIC-8 208 mil, up
to 2.16 mm tall) and an empty PSRAM footprint on its underside, on the
module centreline, so it could not sit flat on the carrier. Measured
on a real module: flash body 15.4 mm from the USB end, PSRAM outline
ending 5.75 mm past it, legs to x +-4.5.

- Pico-Carrier: Edge.Cuts cutout x -5.0..+5.0, y -10.9..+1.6 (footprint
  frame, r 0.5 mm), generated by gen_schematic.py (FLASH_CUTOUT).
  check_library.py asserts it is closed, sized, keeps >=0.5 mm around
  the measured parts and clears every pad by >=0.5 mm. A Pico 2 only
  has bare test pads over it.
- PCB: U1 updated from the library; the seven nets crossing the
  opening (EXP_GP35/43/44/45, HALT_GATE, PICO_P34, GND B.Cu pad 8-33)
  rerouted around it; U1 pads 13/18 back to solid zone connection
  (the library update resets pad overrides). DRC: 0 errors,
  0 unconnected, 35 pre-existing silkscreen warnings. Re-saved by
  KiCad 10.0.6.
- grid_route.py: vias must clear the board edge by their radius, not
  just the track centreline margin (a 0.8 mm via landed 0.0 mm from
  the cutout edge).
- README assembly step and kicad-workflow.md describe the cutout.

Co-Authored-By: Claude Opus 5.5 <noreply@anthropic.com>
Claude-Session: https://claude.ai/code/session_01Bfvc9GBLCYv18x7m3VLkqu
Routing:
- net EXP_GP45: track 45.5 -> 74.9 mm, vias 0 -> 4
- net EXP_GP43: track 46.1 -> 56.5 mm, vias 1 -> 3
- net HALT_GATE: track 48.0 -> 54.3 mm
- net GND: track 552.5 -> 557.8 mm
- net PICO_P34: track 99.0 -> 102.1 mm
- net EXP_GP44: track 44.3 -> 47.2 mm
- net EXP_GP35: track 55.2 -> 57.8 mm
