File: breakout/PiCoCo-Breakout.kicad_pcb (KiCad board)
At the start: 2 copper layers, 52.8 x 99 mm, 7 parts, among them J1 CART_BUS, P1 COCO-CART

Commit message: Added breakout and fab info
Routing:
- net GND: track 146.8 -> 146.3 mm
